Commit message: 添加雷达文件和gazebo控制文件，并修改了launch文件和urdf文件以适应新的雷达和控制配置。增加robot_launch.py文件来启动机器人系统。

File: src/robot_description/urdf/base.xacro (robot description, xacro)
@@ -1,8 +1,8 @@
 <?xml version="1.0"?>
 <robot name="car_robot" xmlns:xacro="http://www.ros.org/wiki/xacro" >
-    <xacro:property name="base_length" value="0.53"/>
+    <xacro:property name="base_length" value="0.66"/>
     <xacro:property name="base_width" value="0.36"/>
     <xacro:property name="base_height" value="0.20"/>
-    <xacro:property name="wheel_radius" value="0.08"/>
+    <xacro:property name="wheel_radius" value="0.10"/>
     <xacro:property name="wheel_width" value="0.03"/>
     <!-- base-link -->
@@ -10,7 +10,5 @@
         <visual>
             <geometry>
-                <geometry>
-                    <sphere radius="0.0001"/>
-                </geometry>
+               <sphere radius="0.0001"/>
             </geometry>
         </visual>
@@ -30,10 +28,10 @@
                     <box size="${base_length} ${base_width} ${base_height}"/>
                 </geometry>
-                <origin xyz="0.0 0.0 ${base_height/2}" rpy="0.0 0.0 0.0"/>
+                <origin xyz="0.0 0.0 0.0" rpy="0.0 0.0 0.0"/>
         </collision>
         <xacro:box_inertia
             m="1.0"
             x="${base_length}" y="${base_width}" z="${base_height}"
-            o_xyz="0.0 0.0 ${base_height/2}"
+            o_xyz="0.0 0.0 0.0"
             o_rpy="0.0 0.0 0.0"/>
     </link>
@@ -52,7 +50,5 @@
             <collision>
                 <geometry>
-                    <geometry>
-                        <sphere radius="${wheel_radius}"/>
-                    </geometry>/>
+                   <sphere radius="${wheel_radius}"/>
                 </geometry>
                 <origin xyz="0.0 0.0 0.0" rpy="1.5708 0.0 0.0"/>
@@ -93,5 +89,5 @@
         <parent link="base_footprint"/>
         <child link="base_link"/>
-        <origin xyz="0.0 0.0 ${(wheel_radius + base_height)/2}" rpy="0.0 0.0 0.0"/>
+        <origin xyz="0.0 0.0 ${wheel_radius + (base_height)/2}" rpy="0.0 0.0 0.0"/>
     </joint>
     <!-- rear_left_wheel_joint -->
@@ -99,5 +95,5 @@
         <parent link="base_link"/>
         <child link="wheel_rear_left"/>
-        <origin xyz="${-(base_length/4)} ${(base_width - wheel_width)/2} -base_height/2" rpy="0.0 0.0 0.0"/>
+        <origin xyz="${-(base_length/4)} ${(base_width - wheel_width)/2} -${base_height/2}" rpy="0.0 0.0 0.0"/>
         <axis xyz="0.0 1.0 0.0"/>
     </joint>
@@ -106,5 +102,5 @@
         <parent link="base_link"/>
         <child link="wheel_rear_right"/>
-        <origin xyz="${-(base_length/4)} ${-(base_width - wheel_width)/2} -base_height/2" rpy="0.0 0.0 0.0"/>
+        <origin xyz="${-(base_length/4)} ${-(base_width - wheel_width)/2} -${base_height/2}" rpy="0.0 0.0 0.0"/>
         <axis xyz="0.0 1.0 0.0"/>
     </joint>
@@ -113,5 +109,5 @@
         <parent link="base_link"/>
         <child link="caster_wheel"/>
-        <origin xyz="${(base_length/4)} 0.0 0.0" rpy="0.0 0.0 0.0"/>
+        <origin xyz="${(base_length/4)} 0.0 -${base_height/2}" rpy="0.0 0.0 0.0"/>
     </joint>
 </robot>

File: src/robot_description/urdf/camera.xacro (robot description, xacro)
@@ -5,5 +5,5 @@
         <visual>
             <geometry>
-                <box size="0.08 0.05 0.03"/>
+                <box size="0.05 0.08 0.03"/>
             </geometry>
             <material name="red">
@@ -14,5 +14,5 @@
         <collision>
             <geometry>
-                <box size="0.08 0.05 0.03"/>
+                <box size="0.05 0.08 0.03"/>
             </geometry>
             <origin xyz="0.0 0.0 0.0" rpy="0.0 0.0 0.0"/>
@@ -20,6 +20,6 @@
         <xacro:box_inertia
             m="1.0"
-            x="0.08"
-            y="0.05"
+            x="0.05"
+            y="0.08"
             z="0.03"
             o_xyz="0.0 0.0 0.0"
@@ -32,3 +32,22 @@
         <origin xyz="${base_length/4} 0.0 ${(base_height +0.03)/2}" rpy="0.0 0.0 0.0"/>
     </joint>
+    <gazebo reference="camera_link">
+        <pose>0 0 0 0 0 0</pose>
+        <visualize>true</visualize>
+        <update_rate>30</update_rate>
+        <topic>/camera/image_raw</topic>
+        <gz_frame_id>camera_link</gz_frame_id>
+        <camera>
+            <horizontal_fov>1.5708</horizontal_fov>
+            <image>
+                <width>640</width>
+                <height>480</height>
+                <format>R8G8B8</format>
+            </image>
+            <clip>
+                <near>0.1</near>
+                <far>100.0</far>
+            </clip>
+        </camera>
+    </gazebo>
 </robot>

File: src/robot_description/urdf/my_robot.urdf.xacro (robot description, xacro)
@@ -4,3 +4,5 @@
     <xacro:include filename="$(find robot_description)/urdf/base.xacro" />
     <xacro:include filename="$(find robot_description)/urdf/camera.xacro"/>
+    <xacro:include filename="$(find robot_description)/urdf/lidar.xacro"/>
+    <xacro:include filename="$(find robot_description)/urdf/gazebo_control.xacro"/>
 </robot>

Commit message: 增加了slam，键盘控制

File: src/robot_description/urdf/base.xacro (robot description, xacro)
@@ -1,4 +1,4 @@
 <?xml version="1.0"?>
-<robot name="car_robot" xmlns:xacro="http://www.ros.org/wiki/xacro" >
+<robot name="my_robot" xmlns:xacro="http://www.ros.org/wiki/xacro" >
     <xacro:property name="base_length" value="0.66"/>
     <xacro:property name="base_width" value="0.36"/>
@@ -50,5 +50,5 @@
             <collision>
                 <geometry>
-                   <sphere radius="${wheel_radius}"/>
+                   <cylinder radius="${wheel_radius}" length="${wheel_width}"/>
                 </geometry>
                 <origin xyz="0.0 0.0 0.0" rpy="1.5708 0.0 0.0"/>
@@ -62,7 +62,9 @@
     </xacro:macro>
     <!-- wheel-links -->
-    <xacro:wheel_link wheel_name="wheel_rear_left"/>
-    <xacro:wheel_link wheel_name="wheel_rear_right"/>
-    <!-- caster_wheel_link -->
+    <xacro:wheel_link wheel_name="left_rear_wheel"/>
+    <xacro:wheel_link wheel_name="right_rear_wheel"/>
+    <xacro:wheel_link wheel_name="left_front_wheel"/>
+    <xacro:wheel_link wheel_name="right_front_wheel"/>
+    <!-- caster_wheel_link
     <link name="caster_wheel">
         <visual>
@@ -84,5 +86,5 @@
             o_xyz="0.0 0.0 0.0"
             o_rpy="1.5708 0.0 0.0"/>
-    </link>
+    </link> -->
     <!-- base_2_footprint_joint -->
     <joint name="base_2_footprint_joint" type="fixed">
@@ -94,5 +96,5 @@
     <joint name="left_rear_wheel_joint" type="continuous">
         <parent link="base_link"/>
-        <child link="wheel_rear_left"/>
+        <child link="left_rear_wheel"/>
         <origin xyz="${-(base_length/4)} ${(base_width - wheel_width)/2} -${base_height/2}" rpy="0.0 0.0 0.0"/>
         <axis xyz="0.0 1.0 0.0"/>
@@ -101,13 +103,27 @@
     <joint name="right_rear_wheel_joint" type="continuous">
         <parent link="base_link"/>
-        <child link="wheel_rear_right"/>
+        <child link="right_rear_wheel"/>
         <origin xyz="${-(base_length/4)} ${-(base_width - wheel_width)/2} -${base_height/2}" rpy="0.0 0.0 0.0"/>
         <axis xyz="0.0 1.0 0.0"/>
     </joint>
-    <!-- caster_wheel_joint -->
+    <!-- front_left_wheel_joint -->
+    <joint name="left_front_wheel_joint" type="continuous">
+        <parent link="base_link"/>
+        <child link="left_front_wheel"/>
+        <origin xyz="${(base_length/4)} ${(base_width - wheel_width)/2} -${base_height/2}" rpy="0.0 0.0 0.0"/>
+        <axis xyz="0.0 1.0 0.0"/>
+    </joint>
+    <!-- front_right_wheel_joint -->
+    <joint name="right_front_wheel_joint" type="continuous">
+        <parent link="base_link"/>
+        <child link="right_front_wheel"/>
+        <origin xyz="${(base_length/4)} ${-(base_width - wheel_width)/2} -${base_height/2}" rpy="0.0 0.0 0.0"/>
+        <axis xyz="0.0 1.0 0.0"/>
+    </joint>
+    <!-- caster_wheel_joint
     <joint name="caster_wheel_joint" type="fixed">
         <parent link="base_link"/>
         <child link="caster_wheel"/>
         <origin xyz="${(base_length/4)} 0.0 -${base_height/2}" rpy="0.0 0.0 0.0"/>
-    </joint>
+    </joint> -->
 </robot>

File: src/robot_description/urdf/camera.xacro (robot description, xacro)
@@ -32,22 +32,3 @@
         <origin xyz="${base_length/4} 0.0 ${(base_height +0.03)/2}" rpy="0.0 0.0 0.0"/>
     </joint>
-    <gazebo reference="camera_link">
-        <pose>0 0 0 0 0 0</pose>
-        <visualize>true</visualize>
-        <update_rate>30</update_rate>
-        <topic>/camera/image_raw</topic>
-        <gz_frame_id>camera_link</gz_frame_id>
-        <camera>
-            <horizontal_fov>1.5708</horizontal_fov>
-            <image>
-                <width>640</width>
-                <height>480</height>
-                <format>R8G8B8</format>
-            </image>
-            <clip>
-                <near>0.1</near>
-                <far>100.0</far>
-            </clip>
-        </camera>
-    </gazebo>
 </robot>

File: src/robot_description/urdf/gazebo_control.xacro (robot description, xacro)
@@ -2,27 +2,106 @@
 <robot xmlns:xacro="http://www.ros.org/wiki/xacro">
     <gazebo>
-        <plugin filename="libgz-sim-diff-drive-system" name="gz::sim::systems::DiffDrive">
+        <plugin filename="gz-sim-diff-drive-system" name="gz::sim::systems::DiffDrive">
             <left_joint>left_rear_wheel_joint</left_joint>
             <right_joint>right_rear_wheel_joint</right_joint>
             <wheel_separation>${base_width - wheel_width}</wheel_separation>
             <wheel_radius>${wheel_radius}</wheel_radius>
-            <update_rate>100.0</update_rate>
             <odom_publish_frequency>10.0</odom_publish_frequency>
-            <topic_name>/cmd_vel</topic_name>
-            <wheel_acceleration>2.0</wheel_acceleration>
-            <wheel_torque>10.0</wheel_torque>
-            <max_linear_speed>2.0</max_linear_speed>
-            <max_angular_speed>1.57</max_angular_speed>
-            <odom_frame_id>/odom</odom_frame_id>
-            <child_frame_id>/base_link</child_frame_id>
+            <topic>/cmd_vel</topic>
             <odom_topic>/odom</odom_topic>
             <tf_topic>/tf</tf_topic>
+            <odom_frame_id>odom</odom_frame_id>
+            <child_frame_id>base_footprint</child_frame_id>
+            <max_linear_velocity>2.0</max_linear_velocity>
+            <min_linear_velocity>-2.0</min_linear_velocity>
+            <max_angular_velocity>1.57</max_angular_velocity>
+            <min_angular_velocity>-1.57</min_angular_velocity>
+            <max_linear_acceleration>2.0</max_linear_acceleration>
+            <min_linear_acceleration>-2.0</min_linear_acceleration>
+            <max_angular_acceleration>3.14</max_angular_acceleration>
+            <min_angular_acceleration>-3.14</min_angular_acceleration>
         </plugin>
-        <plugin filename="libgz-sim-joint-state-publisher" name="gz::sim::systems::JointStatePublisher">
+        <plugin filename="gz-sim-joint-state-publisher" name="gz::sim::systems::JointStatePublisher">
             <joint_name>left_rear_wheel_joint</joint_name>
             <joint_name>right_rear_wheel_joint</joint_name>
             <update_rate>50.0</update_rate>
-            <joint_state_topic>/joint_states</joint_state_topic>
         </plugin>
     </gazebo>
+    <!-- 车身颜色 -->
+    <gazebo reference="base_link">
+        <material>Gazebo/Blue</material>
+    </gazebo>
+    <!-- 轮子颜色 -->
+    <gazebo reference="left_rear_wheel">
+        <material>Gazebo/Green</material>
+        <mu1>1.0</mu1>
+        <mu2>1.0</mu2>
+        <kp>1000000.0</kp>
+        <kd>1.0</kd>
+    </gazebo>
+    <gazebo reference="right_rear_wheel">
+        <material>Gazebo/Green</material>
+        <mu1>1.0</mu1>
+        <mu2>1.0</mu2>
+        <kp>1000000.0</kp>
+        <kd>1.0</kd>
+    </gazebo>
+    <gazebo reference="left_front_wheel">
+        <material>Gazebo/Green</material>
+        <mu1>1.0</mu1>
+        <mu2>1.0</mu2>
+        <kp>1000000.0</kp>
+        <kd>1.0</kd>
+    </gazebo>
+    <gazebo reference="right_front_wheel">
+        <material>Gazebo/Green</material>
+        <mu1>1.0</mu1>
+        <mu2>1.0</mu2>
+        <kp>1000000.0</kp>
+        <kd>1.0</kd>
+    </gazebo>
+    <!-- 相机 -->
+    <gazebo reference="camera_link">
+        <pose>0 0 0 0 0 0</pose>
+        <visualize>true</visualize>
+        <update_rate>30</update_rate>
+        <topic>/camera/image_raw</topic>
+        <gz_frame_id>camera_link</gz_frame_id>
+        <camera>
+            <horizontal_fov>1.5708</horizontal_fov>
+            <image>
+                <width>640</width>
+                <height>480</height>
+                <format>R8G8B8</format>
+            </image>
+            <clip>
+                <near>0.1</near>
+                <far>100.0</far>
+            </clip>
+        </camera>
+    </gazebo>
+    <!-- 雷达 -->
+    <gazebo reference="lidar_link">
+        <sensor type="lidar" name="gpu_lidar">
+            <pose>0 0 0 0 0 0</pose>
+            <visualize>true</visualize>
+            <update_rate>10</update_rate>
+            <topic>/scan</topic>
+            <gz_frame_id>lidar_link</gz_frame_id>
+            <lidar>
+                <scan>
+                    <horizontal>
+                        <samples>720</samples>
+                        <min_angle>-3.14</min_angle>
+                        <max_angle>3.14</max_angle>
+                    </horizontal>
+                </scan>
+                <range>
+                    <min>0.1</min>
+                    <max>10.0</max>
+                    <resolution>0.01</resolution>
+                </range>
+            </lidar>
+        </sensor>
+    </gazebo>
 </robot>

File: src/robot_description/urdf/lidar.xacro (robot description, xacro)
@@ -33,26 +33,3 @@
         <origin xyz="${-(base_length/4)} 0.0 ${(base_height + lidar_length)/2}" rpy="0.0 0.0 0.0"/>
     </joint>
-    <gazebo reference="lidar_link">
-        <sensor type="lidar" name="gpu_lidar">
-            <pose>0 0 0 0 0 0</pose>
-            <visualize>true</visualize>
-            <update_rate>10</update_rate>
-            <topic>/scan</topic>
-            <gz_frame_id>lidar_link</gz_frame_id>
-            <lidar>
-                <scan>
-                    <horizontal>
-                        <samples>720</samples>
-                        <min_angle>-3.14</min_angle>
-                        <max_angle>3.14</max_angle>
-                    </horizontal>
-                </scan>
-                <range>
-                    <min>0.1</min>
-                    <max>10.0</max>
-                    <resolution>0.01</resolution>
-                </range>
-            </lidar>
-        </sensor>
-    </gazebo>
 </robot>

Commit message: 小车tf_tree正常了

File: src/robot_description/urdf/base.xacro (robot description, xacro)
@@ -88,5 +88,5 @@
     </link> -->
     <!-- base_2_footprint_joint -->
-    <joint name="base_2_footprint_joint" type="fixed">
+    <joint name="base_footprint_joint" type="fixed">
         <parent link="base_footprint"/>
         <child link="base_link"/>

File: src/robot_description/urdf/gazebo_control.xacro (robot description, xacro)
@@ -11,5 +11,8 @@
             <odom_topic>/odom</odom_topic>
             <tf_topic>/tf</tf_topic>
-            <odom_frame_id>odom</odom_frame_id>
+            <!-- 此处不是odom_frame_id,否则不能发布odom话题，tf_tree上没有odom，如果使用odom_frame_id,
+            则这个标签不起作用，系统会使用默认的odom话题，并给他加上命名空间，这个命名空间会和my_robot.urdf.xacro
+            文件中的robot标签 中的name属性值一样-->
+            <frame_id>odom</frame_id>
             <child_frame_id>base_footprint</child_frame_id>
             <max_linear_velocity>2.0</max_linear_velocity>
@@ -77,21 +80,23 @@
     <!-- 相机 -->
     <gazebo reference="camera_link">
-        <pose>0 0 0 0 0 0</pose>
-        <visualize>true</visualize>
-        <update_rate>30</update_rate>
-        <topic>/camera/image_raw</topic>
-        <gz_frame_id>camera_link</gz_frame_id>
-        <camera>
-            <horizontal_fov>1.5708</horizontal_fov>
-            <image>
-                <width>640</width>
-                <height>480</height>
-                <format>R8G8B8</format>
-            </image>
-            <clip>
-                <near>0.1</near>
-                <far>100.0</far>
-            </clip>
-        </camera>
+        <sensor name='camera' type='camera'>
+            <pose>0 0 0 0 0 0</pose>
+            <visualize>true</visualize>
+            <update_rate>30</update_rate>
+            <topic>/camera/image_raw</topic>
+            <gz_frame_id>camera_link</gz_frame_id>
+            <camera>
+                <horizontal_fov>1.5708</horizontal_fov>
+                <image>
+                    <width>640</width>
+                    <height>480</height>
+                    <format>R8G8B8</format>
+                </image>
+                <clip>
+                    <near>0.1</near>
+                    <far>100.0</far>
+                </clip>
+            </camera>
+        </sensor>
     </gazebo>
     <!-- 雷达 -->

File: src/robot_description/urdf/lidar.xacro (robot description, xacro)
@@ -11,5 +11,5 @@
             o_xyz="0.0 0.0 0.0"
             o_rpy="0.0 0.0 0.0"/>
-        <visual name="">
+        <visual >
             <origin xyz="0.0 0.0 0.0" rpy="0.0 0.0 0.0"/>
             <geometry>

File: src/robot_description/urdf/my_robot.urdf.xacro (robot description, xacro)
@@ -1,5 +1,5 @@
 <?xml version="1.0"?>
 <!-- 这个文文件的robot标签一定要有name属性，否则rviz和gazebo都不能加载机器人 -->
-<robot name="firstrobot" xmlns:xacro="http://www.ros.org/wiki/xacro" >
+<robot name="first_robot" xmlns:xacro="http://www.ros.org/wiki/xacro" >
     <xacro:include filename="$(find robot_description)/urdf/common_macro.xacro" />
     <xacro:include filename="$(find robot_description)/urdf/base.xacro" />
