Commit message: 增加rviz启动参数

File: src/robot_description/urdf/base.xacro (robot description, xacro)
@@ -1,9 +1,9 @@
 <?xml version="1.0"?>
 <robot xmlns:xacro="http://www.ros.org/wiki/xacro" >
-    <xacro:property name="base_length" value="0.66"/>
-    <xacro:property name="base_width" value="0.36"/>
+    <xacro:property name="base_length" value="0.25"/>
+    <xacro:property name="base_width" value="0.25"/>
     <xacro:property name="base_height" value="0.20"/>
-    <xacro:property name="wheel_radius" value="0.10"/>
-    <xacro:property name="wheel_width" value="0.03"/>
+    <xacro:property name="wheel_radius" value="0.032"/>
+    <xacro:property name="wheel_width" value="0.04"/>
     <!-- base-link -->
     <link name="base_footprint">
