Commit message: 增加imu和修正相机

File: src/robot_description/urdf/camera.xacro (robot description, xacro)
@@ -30,5 +30,5 @@
         <parent link="base_link"/>
         <child link="camera_link"/>
-        <origin xyz="${base_length/4} 0.0 ${(base_height +0.03)/2}" rpy="0.0 0.0 0.0"/>
+        <origin xyz="${base_length/2 - 0.025} 0.0 ${(base_height +0.03)/2}" rpy="0.0 0.0 0.0"/>
     </joint>
 </robot>

File: src/robot_description/urdf/gazebo_control.xacro (robot description, xacro)
@@ -58,26 +58,4 @@
         <mu2>0.000001</mu2>
     </gazebo>
-    <!-- 相机 -->
-    <gazebo reference="camera_link">
-        <sensor name='camera' type='camera'>
-            <pose>0 0 0 0 0 0</pose>
-            <visualize>true</visualize>
-            <update_rate>30</update_rate>
-            <topic>/camera/image_raw</topic>
-            <gz_frame_id>camera_link</gz_frame_id>
-            <camera>
-                <horizontal_fov>1.5708</horizontal_fov>
-                <image>
-                    <width>640</width>
-                    <height>480</height>
-                    <format>R8G8B8</format>
-                </image>
-                <clip>
-                    <near>0.1</near>
-                    <far>100.0</far>
-                </clip>
-            </camera>
-        </sensor>
-    </gazebo>
     <!-- 雷达 -->
     <gazebo reference="lidar_link">
@@ -104,3 +82,49 @@
         </sensor>
     </gazebo>
+    <!-- 相机 -->
+    <gazebo reference="camera_link">
+         <sensor name="camera" type="camera">
+        <always_on>true</always_on>
+        <update_rate>30</update_rate>
+        <topic>/camera/image_raw</topic>
+        <camera>
+            <horizontal_fov>1.047</horizontal_fov>
+            <image>
+                <width>640</width>
+                <height>480</height>
+                <format>R8G8B8</format>
+            </image>
+            <clip>
+                <near>0.05</near>
+                <far>8.0</far>
+            </clip>
+            <noise>
+                <type>gaussian</type>
+                <mean>0.0</mean>
+                <stddev>0.007</stddev>
+            </noise>
+        </camera>
+        </sensor>
+    </gazebo>
+    <!-- imu -->
+    <gazebo reference="imu_link">
+        <sensor name="imu_senser" type="imu">
+            <update_rate>50.0</update_rate>
+            <topic>/imu</topic>
+            <always_on>true</always_on>
+            <visualize>true</visualize>
+            <imu>
+            <angular_velocity>
+                <x><noise type="gaussian"><stddev>0.01</stddev></noise></x>
+                <y><noise type="gaussian"><stddev>0.01</stddev></noise></y>
+                <z><noise type="gaussian"><stddev>0.01</stddev></noise></z>
+            </angular_velocity>
+            <linear_acceleration>
+                <x><noise type="gaussian"><stddev>0.1</stddev></noise></x>
+                <y><noise type="gaussian"><stddev>0.1</stddev></noise></y>
+                <z><noise type="gaussian"><stddev>0.1</stddev></noise></z>
+            </linear_acceleration>
+        </imu>
+        </sensor>
+    </gazebo>
 </robot>

File: src/robot_description/urdf/my_robot.urdf.xacro (robot description, xacro)
@@ -7,3 +7,4 @@
     <xacro:include filename="$(find robot_description)/urdf/lidar.xacro"/>
     <xacro:include filename="$(find robot_description)/urdf/gazebo_control.xacro"/>
+    <xacro:include filename="$(find robot_description)/urdf/imu.xacro"/>
 </robot>
