Commit message: 换了world文件，可以建图了

File: src/robot_description/urdf/gazebo_control.xacro (robot description, xacro)
@@ -60,6 +60,6 @@
     <gazebo reference="left_front_wheel">
         <material>Gazebo/Green</material>
-        <mu1>0.0</mu1>
-        <mu2>0.0</mu2>
+        <mu1>1.0</mu1>
+        <mu2>1.0</mu2>
         <kp>10000000.0</kp>
         <kd>1.0</kd>
@@ -70,6 +70,6 @@
     <gazebo reference="right_front_wheel">
         <material>Gazebo/Green</material>
-        <mu1>0.0</mu1>
-        <mu2>0.0</mu2>
+        <mu1>1.0</mu1>
+        <mu2>1.0</mu2>
         <kp>10000000.0</kp>
         <kd>1.0</kd>
@@ -105,5 +105,5 @@
             <pose>0 0 0 0 0 0</pose>
             <visualize>true</visualize>
-            <update_rate>10</update_rate>
+            <update_rate>5</update_rate>
             <topic>/scan</topic>
             <gz_frame_id>lidar_link</gz_frame_id>
@@ -118,5 +118,5 @@
                 <range>
                     <min>0.1</min>
-                    <max>10.0</max>
+                    <max>20.0</max>
                     <resolution>0.01</resolution>
                 </range>

File: src/robot_description/urdf/lidar.xacro (robot description, xacro)
@@ -31,5 +31,5 @@
         <parent link="base_link"/>
         <child link="lidar_link"/>
-        <origin xyz="${-(base_length/4)} 0.0 ${(base_height + lidar_length)/2}" rpy="0.0 0.0 0.0"/>
+        <origin xyz="0.0 0.0 ${(base_height/2 + lidar_length/2 + 0.1)}" rpy="0.0 0.0 0.0"/>
     </joint>
 </robot>

Commit message: 把导航功能加到总的启动文件里，并通过延迟navigation启动修复rviz不加载地图问题

File: src/robot_description/urdf/gazebo_control.xacro (robot description, xacro)
@@ -21,5 +21,5 @@
             <min_angular_velocity>-1.57</min_angular_velocity>
             <max_linear_acceleration>2.0</max_linear_acceleration>
-            <min_linear_acceleration>-2.0</min_linear_acceleration>
+            <min_linear_acceleration>-5.0</min_linear_acceleration>
             <max_angular_acceleration>3.14</max_angular_acceleration>
             <min_angular_acceleration>-3.14</min_angular_acceleration>
@@ -111,20 +111,13 @@
         <sensor name="imu_senser" type="imu">
             <update_rate>50.0</update_rate>
+            <visualize>true</visualize>
+            <always_on>1</always_on>
+            <visualize>true</visualize>
             <topic>/imu</topic>
-            <always_on>true</always_on>
-            <visualize>true</visualize>
-            <imu>
-            <angular_velocity>
-                <x><noise type="gaussian"><stddev>0.01</stddev></noise></x>
-                <y><noise type="gaussian"><stddev>0.01</stddev></noise></y>
-                <z><noise type="gaussian"><stddev>0.01</stddev></noise></z>
-            </angular_velocity>
-            <linear_acceleration>
-                <x><noise type="gaussian"><stddev>0.1</stddev></noise></x>
-                <y><noise type="gaussian"><stddev>0.1</stddev></noise></y>
-                <z><noise type="gaussian"><stddev>0.1</stddev></noise></z>
-            </linear_acceleration>
-        </imu>
         </sensor>
     </gazebo>
+    <gazebo>
+      <plugin filename="gz-sim-imu-system" name="gz::sim::systems::Imu">
+      </plugin>
+    </gazebo>
 </robot>

File: src/robot_description/urdf/imu.xacro (robot description, xacro)
@@ -19,8 +19,8 @@
         o_rpy="0.0 0.0 0.0"/>
     </link>
-    <joint name="imu_joint" type="fixed">
-        <parent link="base_link"/>
-        <child link="imu_link"/>
-        <origin xyz="0 0 0.05" rpy="0 0 0"/>
+    <joint name="imu_to_base_link" type="fixed">
+      <parent link="base_link"/>
+      <child link="imu_link"/>
+      <origin xyz="0 0 0" rpy="0 0 0"/>
     </joint>
 </robot>
